Commit message: added mobile base to robots

File: examples/06-panda_guidance/panda_arm.urdf (robot description, URDF)
Before this commit: robot panda, 8 links, 7 joints
Links:
- added link platform0, mass 4
- added link platform1, mass 4
- link link0: geometry visual mesh filename=../../../../examples/models/franka_panda/meshes/visual/link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
- link link1: geometry visual mesh filename=../../../../examples/models/franka_panda/meshes/visual/link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
- link link2: geometry collision mesh filename=../../../../examples/models/panda/meshes/link2.obj; visual mesh filename=../../../../examples/models/franka_panda/meshes/visual/link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
- link link3: geometry collision mesh filename=../../../../examples/models/panda/meshes/link3.obj; visual mesh filename=../../../../examples/models/franka_panda/meshes/visual/link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
- link link4: geometry collision mesh filename=../../../../examples/models/panda/meshes/link4.obj; visual mesh filename=../../../../examples/models/franka_panda/meshes/visual/link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
- link link5: geometry collision mesh filename=../../../../examples/models/panda/meshes/link5.obj; visual mesh filename=../../../../examples/models/franka_panda/meshes/visual/link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
- link link6: geometry collision mesh filename=../../../../examples/models/panda/meshes/link6.obj; visual mesh filename=../../../../examples/models/franka_panda/meshes/visual/link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
- link link7: geometry collision mesh filename=../../../../examples/models/panda/meshes/link7.obj; visual mesh filename=../../../../examples/models/franka_panda/meshes/visual/link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
Joints:
- added joint xTrans: type prismatic, parent platform0, child platform1, origin xyz=0 0 0 rpy=0 0 0, axis 1 0 0, limit lower=-2.8973 upper=2.8973 effort=12 velocity=2.6100
- added joint yTrans: type prismatic, parent platform1, child link0, origin xyz=0 0 0 rpy=0 0 0, axis 0 1 0, limit lower=-2.8973 upper=2.8973 effort=12 velocity=2.6100
