Commit message: Attempting to implement momentum-based observer

File: build_qt/examples/06-panda_guidance/resources/panda_arm.urdf (robot description, URDF)
Before this commit: robot panda, 8 links, 7 joints
Links:
- link link0: geometry visual mesh filename=../../../../examples/models/panda/meshes/link0.obj
- link link1: geometry visual mesh filename=../../../../examples/models/panda/meshes/link1.obj

Commit message: Collision spheres and active following guidelines added. Debugging collision detection with payload.

File: build_qt/examples/06-panda_guidance/resources/panda_arm.urdf (robot description, URDF)
Before this commit: robot panda, 10 links, 9 joints
Links:
- link link0: geometry visual mesh filename=../../../../examples/models/panda/meshes/link0.obj
- link link1: geometry visual mesh filename=../../../../examples/models/panda/meshes/link1.obj
- link link2: geometry collision mesh filename=../../../../examples/models/panda/meshes/link2.obj; visual mesh filename=../../../../examples/models/panda/meshes/link2.obj
- link link3: geometry collision mesh filename=../../../../examples/models/panda/meshes/link3.obj; visual mesh filename=../../../../examples/models/panda/meshes/link3.obj
- link link4: geometry collision mesh filename=../../../../examples/models/panda/meshes/link4.obj; visual mesh filename=../../../../examples/models/panda/meshes/link4.obj
- link link5: geometry collision mesh filename=../../../../examples/models/panda/meshes/link5.obj; visual mesh filename=../../../../examples/models/panda/meshes/link5.obj
- link link6: geometry collision mesh filename=../../../../examples/models/panda/meshes/link6.obj; visual mesh filename=../../../../examples/models/panda/meshes/link6.obj
- link link7: geometry collision mesh filename=../../../../examples/models/panda/meshes/link7.obj; visual mesh filename=../../../../examples/models/panda/meshes/link7.obj
